File: PLC4UNI/plc/kicad diseño/PLC Electiva/PLC Electiva.kicad_sch (KiCad schematic)
At the start: 0 parts

Commit message: Esquemático actualizádo
Parts:
- added connector-down1, connector-down2, connector-up1, connector-up2: Screw_Terminal_9_P5.00mm, TerminalBlock_Phoenix:TerminalBlock_Phoenix_PT-1,5-9-5.0-H_1x09_P5.00mm_Horizontal, symbol PCM_SL_Screw_Terminal:Screw_Terminal_9_P5.00mm
Connections:
- net main/CON-IN-4-20MA_1: now also connector-up2.6
- net main/CON-IN-4-20MA_2: now also connector-up2.5
- net main/CON-IN_CT_N: now also connector-up2.4
- net main/CON-IN_CT_P: now also connector-up2.3
- net main/CON-IN_VAC_P: now also connector-up2.1
- net main/CON_IN_0-10V_1: now also connector-up2.8
- net main/CON_IN_0-10V_2: now also connector-up2.7
- net main/CON_IN_NPN1: now also connector-up1.7
- net main/CON_IN_NPN2: now also connector-up1.6
- net main/CON_IN_NPN3: now also connector-up1.5
- net main/CON_IN_NPN4: now also connector-up1.4
- net main/CON_IN_PNP1: now also connector-up1.3
- net main/CON_IN_PNP2: now also connector-up1.2
- net main/CON_IN_TC+: now also connector-up1.1
- net main/CON_IN_TC-: now also connector-up2.9
- net main/CON_OUT_0-10V: now also connector-down2.8
- net main/CON_OUT_4-20MA: now also connector-down2.7
- net main/CON_OUT_NPN1: now also connector-down1.4
- net main/CON_OUT_NPN2: now also connector-down1.5
- net main/CON_OUT_NPN3: now also connector-down1.6
- net main/CON_OUT_NPN4: now also connector-down1.7
- net main/CON_OUT_PNP1: now also connector-down1.8
- net main/CON_OUT_PNP2: now also connector-down1.9
- net main/CON_OUT_RLY1_COM: now also connector-down2.1
- net main/CON_OUT_RLY1_NC: now also connector-down2.2
- net main/CON_OUT_RLY1_NO: now also connector-down2.3
- net main/CON_OUT_RLY2_COM: now also connector-down2.6
- net main/CON_OUT_RLY2_NC: now also connector-down2.4
- net main/CON_OUT_RLY2_NO: now also connector-down2.5
- net main/CON_RS485_A: now also connector-down1.2
- net main/CON_RS485_B: now also connector-down1.3
- net main/CON_RS485_G: now also connector-down1.1
- new net +24V: connector-up1.9
- new net Earth: connector-up2.2
- new net GND: connector-down2.9, connector-up1.8
Other:
- added sheet Josue Herrera (josueherrera.kicad_sch)
