File: PLC4UNI/plc/kicad diseño/PLC Electiva/control.kicad_sch (KiCad schematic)
At the start: 0 parts

Commit message: Esquemático actualizádo
Parts:
- added C13: 100NF, Capacitor_SMD_AKL:C_0603_1608Metric, symbol Capacitor_AKL:C_0603
- added C25: 100nf, Capacitor_SMD_AKL:C_0603_1608Metric, symbol Capacitor_AKL:C_0603
- added C26: 1uF, Capacitor_SMD_AKL:C_0603_1608Metric, symbol Capacitor_AKL:C_0603
- added D17, D18, D19, D20, D21: ESD5Z3.3T, Diode_SMD_AKL:D_SOD-523, symbol Diode_TVS_AKL:ESD5Z3.3T
- added J1: Conn_02x08_Odd_Even, Connector_PinHeader_2.54mm:PinHeader_2x08_P2.54mm_Vertical, symbol Connector_Generic:Conn_02x08_Odd_Even
- added LED5: LED_0603_Red, LED_SMD_AKL:LED_0603_1608Metric, symbol LED_AKL:LED_0603_Red
- added R30, R31: R_0603, Resistor_SMD_AKL:R_0603_1608Metric, symbol Resistor_US_AKL:R_0603
- added R4: 22K, Resistor_SMD_AKL:R_0603_1608Metric, symbol Resistor_US_AKL:R_0603
- added R50: 2.2K, Resistor_SMD_AKL:R_0603_1608Metric, symbol Resistor_US_AKL:R_0603
- added SW1: TS-1088-AR02016, EasyEDA:SW-SMD_L3.9-W3.0-P4.45, symbol EasyEDA:TS-1088-AR02016
- added TP1, TP2, TP3, TP4: TestPoint_Hole1, 4ms_TestPoint:TestPoint_WireHole, symbol MG_ELECTROMECANICAL:TestPoint_Hole1
- added U1: ESP32-S3-WROOM-1, RF_Module:ESP32-S3-WROOM-1U, symbol RF_Module:ESP32-S3-WROOM-1
- added U10: ADS1115IDGS, Package_SO:TSSOP-10_3x3mm_P0.5mm, symbol Analog_ADC:ADS1115IDGS
- added U4: RS485-PROTECT, MG_footprints:RS-485-PROTECT, symbol MG_CONNECTORS:RS485-PROTECT
Connections:
- new net: LED5.2 (A), R50.1
- new net +24V: R30.1
- new net +3.3V: C13.1, J1.2 (Pin_2), R4.2, U1.2 (3V3), U10.8 (VDD), U4.1 (VCC)
- new net +5V: J1.1 (Pin_1)
- new net CON_RS485_A: U4.7 (A)
- new net CON_RS485_B: U4.8 (B)
- new net CON_RS485_G: U4.6 (RGND)
- new net EMRX: U1.36 (RXD0)
- new net EM_TX: U1.37 (TXD0)
- new net EN: C26.2, D17.1 (K), R4.1, SW1.1, U1.3 (EN)
- new net GND: C13.2, C25.2, C26.1, D17.2 (A), D18.2 (A), D19.2 (A), D20.2 (A), D21.2 (A), J1.15 (Pin_15), J1.16 (Pin_16), LED5.1 (K), R31.2, SW1.2, U1.1 (GND), U1.40 (GND), U1.41 (GND), U10.1 (ADDR), U10.3 (GND), U4.2 (GND)
- new net GPIO1: U1.8 (IO15)
- new net GPIO2: U1.9 (IO16)
- new net I2C_SCK: J1.10 (Pin_10)
- new net I2C_SDA: J1.8 (Pin_8)
- new net IN-0-10V/OUT3V: TP3.1, U10.6 (AIN2)
- new net IN-0-10V1/OUT3V: TP4.1, U10.7 (AIN3)
- new net IN-4-20MA/OUT: TP1.1, U10.4 (AIN0)
- new net IN-4-20MA1/OUT: TP2.1, U10.5 (AIN1)
- new net IN_NPN1: U1.27 (IO0)
- new net IN_NPN2: U1.39 (IO1)
- new net IN_NPN3: U1.38 (IO2)
- new net IN_NPN4: U1.15 (IO3)
- new net IN_PNP1: U1.4 (IO4)
- new net IN_PNP2: U1.5 (IO5)
- new net IN_VDC_ADC: C25.1, R30.2, R31.1, U1.6 (IO6)
- new net LCD_CS: J1.13 (Pin_13)
- new net LCD_EN: J1.12 (Pin_12)
- new net LED_INFO: R50.2, U1.23 (IO21)
- new net OUT_NPN1: U1.31 (IO38)
- new net OUT_NPN2: U1.32 (IO39)
- new net OUT_NPN3: U1.33 (IO40)
- new net OUT_NPN4: U1.34 (IO41)
- new net OUT_PNP1: U1.16 (IO46)
- new net OUT_PNP2: U1.24 (IO47)
- new net OUT_RLY1: U1.35 (IO42)
- new net OUT_RLY2: U1.26 (IO45)
- new net RESET: J1.11 (Pin_11)
- new net RS485-CON: U4.5 (CON)
- new net RS485-RX: U4.4 (RXD)
- new net RS485-TX: U4.3 (TXD)
- new net SD_CS: D21.1 (K), J1.3 (Pin_3)
- new net SPI_CLK: D18.1 (K), J1.9 (Pin_9)
- new net SPI_MISO: D19.1 (K), J1.7 (Pin_7)
- new net SPI_MOSI: D20.1 (K), J1.5 (Pin_5)
- new net TEMP_CS: U1.25 (IO48)
- new net TP_INT: J1.14 (Pin_14)
- new net USB+: J1.4 (Pin_4)
- new net USB-: J1.6 (Pin_6)
- new net acc_cs: U1.7 (IO7)
- new net clk: U1.22 (IO14)
- new net cs: U1.19 (IO11)
- new net i2c_scl: U1.11 (IO18), U10.10 (SCL)
- new net i2c_sda: U1.10 (IO17), U10.9 (SDA)
- new net miso: U1.20 (IO12)
- new net mosi: U1.21 (IO13)
- new net rs485-com: U1.18 (IO10)
- new net rs485_rx: U1.12 (IO8)
- new net rs485_tx: U1.17 (IO9)
- new net usb+: U1.14 (USB_D+)
- new net usb-: U1.13 (USB_D-)
- no-connect marks 0 -> 3
Other:
- added sheet EnergyMeterA1 (EnergyMeterA1.kicad_sch)
- added sheet IN-0-10V (IN-0-10V.kicad_sch)
- added sheet IN-0-10V1 (IN-0-10V.kicad_sch)
- added sheet IN-4-20MA (IN-4-20MA.kicad_sch)
- added sheet IN-4-20MA1 (IN-4-20MA.kicad_sch)
- added sheet IN-DI (IN-DI.kicad_sch)
- added sheet IN-DI1 (IN-DI.kicad_sch)
- added sheet IN-DI2 (IN-DI.kicad_sch)
- added sheet IN-DI3 (IN-DI.kicad_sch)
- added sheet IN-DI4 (IN-DI.kicad_sch)
- added sheet IN-DI5 (IN-DI.kicad_sch)
- added sheet OUT-0-10V (OUT-0-10V.kicad_sch)
- added sheet OUT-4-20MA (OUT-4-20MA.kicad_sch)
- added sheet OUT-NPN (OUT-NPN.kicad_sch)
- added sheet OUT-NPN1 (OUT-NPN.kicad_sch)
- added sheet OUT-NPN2 (OUT-NPN.kicad_sch)
- added sheet OUT-NPN3 (OUT-NPN.kicad_sch)
- added sheet OUT-PNP (OUT-PNP.kicad_sch)
- added sheet RLY (RLY.kicad_sch)
- added sheet TC (TC.kicad_sch)
